File: LCD_HAT/LCD_HAT.kicad_sch (KiCad schematic)
At the start: 8 parts, among them J1 Qwiic, J2 LCD, SW1 SW_Push, SW2 SW_Push

Commit message: Updated project files
Parts:
- added J3, J4: PWR_JUMPER, Connector_PinHeader_2.54mm:PinHeader_1x02_P2.54mm_Vertical, symbol Connector:Conn_01x02_Pin
- added R3: 68K, Resistor_SMD:R_0603_1608Metric, symbol Device:R
Connections:
- net +3.3V: now also J3.2 (Pin_2), J4.2 (Pin_2), R3.1; no longer J1.3 (Pin_3), J2.2 (Pin_2)
- net GND: now also J1.1 (Pin_1); no longer J1.4 (Pin_4)
- net at A1.21 (D2), A2.5 (D2), J2.5 (Pin_5): now also R3.2
- net at A1.17 (SDA), A2.23 (A4): now also J1.3 (Pin_3); no longer J1.2 (Pin_2)
- net at A1.18 (SCL), A2.24 (A5): now also J1.4 (Pin_4); no longer J1.1 (Pin_1)
- new net: J2.2 (Pin_2), J3.1 (Pin_1)
- new net: J1.2 (Pin_2), J4.1 (Pin_1)
Other:
- note added: "Pull-up for RESET line of LCD"
