File: ds3231_plus/ds3231_plus.kicad_pcb (KiCad board)
At the start: 2 copper layers, 18 x 22 mm, 11 parts, among them J2 Conn_01x05_Female

Commit message: Updated project files
Parts:
- removed Backup Battery: 3.0, Battery:BatteryHolder_Keystone_2998_1x6.8mm
- added BT1: 3.0, Battery:CR44_Tabs, B.Cu at (142.2, 89.5)
- SW1: renamed from Battery Cutoff
- renumbered Qwiic to QWIIC, J2 to RPI1, DS3231 to U1
Connections:
- QWIIC pad 1: /SCL -> GND
- QWIIC pad 2: /SDA -> +3.3V
- QWIIC pad 3: +3.3V -> /SDA
- QWIIC pad 4: GND -> /SCL
Routing:
- net Net-(BT1-+): track 19.5 -> 6.08 mm
- net GND: track 32.5 -> 26.3 mm, vias 3 -> 4
- net +3.3V: track 47.1 -> 42.2 mm
- net /SCL: track 28.2 -> 24.0 mm
- net /SDA: track 21.6 -> 23.4 mm
Other:
- board size 18 x 22 mm -> 18.2 x 22.2 mm
