File: ds3231_plus/ds3231_plus.kicad_sch (KiCad schematic)
At the start: 10 parts, among them J1 Conn_01x04_Female, J2 Conn_01x05_Female, SW1 SW_DIP_x01, U1 DS3231M

Commit message: Updated project files
Parts:
- BT1: footprint Battery:BatteryHolder_Keystone_2998_1x6.8mm -> Battery:CR44_Tabs
- renumbered J1 to QWIIC1, J2 to RPI1
Connections:
- net +3.3V: now also QWIIC1.2 (Pin_2); no longer QWIIC1.3 (Pin_3)
- net GND: now also QWIIC1.1 (Pin_1); no longer QWIIC1.4 (Pin_4)
- net SCL: now also QWIIC1.4 (Pin_4); no longer QWIIC1.1 (Pin_1)
- net SDA: now also QWIIC1.3 (Pin_3); no longer QWIIC1.2 (Pin_2)
